Commit message: Update robot_urdf.urdf

File: urdf/robot.urdf.urdf (robot description, URDF)
Before this commit: robot robot.urdf, 5 links, 4 joints
Links:
- link base_link: geometry collision mesh filename=package://robot_description/meshes/base_link.STL; visual mesh filename=package://robot_description/meshes/base_link.STL
- link caster_wheel: geometry collision mesh filename=package://robot_description/meshes/caster_wheel.STL; visual mesh filename=package://robot_description/meshes/caster_wheel.STL
- link left_wheel: geometry collision mesh filename=package://robot_description/meshes/left_wheel.STL; visual mesh filename=package://robot_description/meshes/left_wheel.STL
- link link_ydlidar: geometry collision mesh filename=package://robot_description/meshes/link_ydlidar.STL; visual mesh filename=package://robot_description/meshes/link_ydlidar.STL
- link right_wheel: geometry collision mesh filename=package://robot_description/meshes/right_wheel.STL; visual mesh filename=package://robot_description/meshes/right_wheel.STL
